File: kicad/zusatzsignal-2-led/zusatzsignal.kicad_pcb (KiCad board)
At the start: 2 copper layers, 3.7 x 5.3 mm, 4 parts

Commit message: MSv2
Parts:
- removed D2: LED, LED_SMD:LED_0603_1608Metric
- removed G, V: SolderWirePad_1x01_SMD_1x2mm, Connector_Wire:SolderWirePad_1x01_SMD_1x2mm
- added J1: VCC, Connector_Wire:SolderWirePad_1x01_SMD_1x2mm, B.Cu at (140.7, 80.7)
- added J2: Zs, Connector_Wire:SolderWirePad_1x01_SMD_1x2mm, B.Cu at (139.0, 80.7)
- moved D1 0.91 mm to (139.9, 81.6)
Connections:
- D1 pad 2: VCC -> Net-(D1-Pad2)
Routing:
- net VCC: track 4.38 -> 0.00 mm, vias 1 -> 0
- net Net-(D1-Pad2): track 0.00 -> 3.63 mm, vias 0 -> 1
- net GND: track 3.24 -> 0.00 mm, vias 1 -> 0
- net Net-(D1-Pad1): track 1.76 -> 3.40 mm, vias 0 -> 1
Other:
- board text added: "+"
