File: kicad/Mehrabschnittssignal/Mehrabschnittssignal.kicad_sch (KiCad schematic)
At the start: 19 parts, among them J0 VCC, J1 VkzBw, J2 ROT, J3 GELB, J4 GRÜN, J5 Zs7-3, J6 Ra, J7 Zs7-1, J8 Zs7-2, J9 Ra/Zs1

Commit message: Update MS README
Parts:
- J0, J1, J2, J3, J4, J5, J6, J7, J8, J9: now left out of the parts list
Other:
- moved on the sheet: J0
Changed lines of the file:
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@@
     (stroke (width 0) (type default) (color 0 0 0 0))
   )
-  (wire (pts (xy 71.12 59.69) (xy 78.74 59.69))
+  (wire (pts (xy 69.85 59.69) (xy 78.74 59.69))
     (stroke (width 0) (type default) (color 0 0 0 0))
   )
@@
   )
   (symbol (lib_id "Connector:Conn_01x01_Male") (at 64.77 100.33 0) (unit 1)
-    (in_bom yes) (on_board yes)
+    (in_bom no) (on_board yes)
     (property "Reference" "J9" (id 0) (at 62.23 100.33 0))
     (property "Value" "Ra/Zs1" (id 1) (at 55.88 100.33 0))
@@
   )
   (symbol (lib_id "Connector:Conn_01x01_Male") (at 64.77 92.71 0) (unit 1)
-    (in_bom yes) (on_board yes)
+    (in_bom no) (on_board yes)
     (property "Reference" "J7" (id 0) (at 62.23 92.71 0))
     (property "Value" "Zs7-1" (id 1) (at 55.88 92.71 0))
@@
   )
   (symbol (lib_id "Connector:Conn_01x01_Male") (at 64.77 96.52 0) (unit 1)
-    (in_bom yes) (on_board yes)
+    (in_bom no) (on_board yes)
     (property "Reference" "J8" (id 0) (at 62.23 96.52 0))
     (property "Value" "Zs7-2" (id 1) (at 55.88 96.52 0))
@@
   )
   (symbol (lib_id "Connector:Conn_01x01_Male") (at 64.77 69.85 0) (unit 1)
-    (in_bom yes) (on_board yes)
+    (in_bom no) (on_board yes)
     (property "Reference" "J1" (id 0) (at 62.23 69.85 0))
     (property "Value" "VkzBw" (id 1) (at 55.88 69.85 0))
@@
   )
   (symbol (lib_id "Connector:Conn_01x01_Male") (at 64.77 88.9 0) (unit 1)
-    (in_bom yes) (on_board yes)
+    (in_bom no) (on_board yes)
     (property "Reference" "J6" (id 0) (at 62.23 88.9 0))
     (property "Value" "Ra" (id 1) (at 55.88 88.9 0))
@@
     (pin "1")
   )
-  (symbol (lib_id "Connector:Conn_01x01_Male") (at 66.04 59.69 0) (unit 1)
-    (in_bom yes) (on_board yes)
-    (property "Reference" "J0" (id 0) (at 63.5 59.69 0))
-    (property "Value" "VCC" (id 1) (at 57.15 59.69 0))
-    (property "Footprint" "Connector_Wire:SolderWirePad_1x01_SMD_1x2mm" (id 2) (at 66.04 59.69 0)
-      (effects (font (size 1.27 1.27)) hide)
-    )
-    (property "Datasheet" "~" (id 3) (at 66.04 59.69 0)
+  (symbol (lib_id "Connector:Conn_01x01_Male") (at 64.77 59.69 0) (unit 1)
+    (in_bom no) (on_board yes)
+    (property "Reference" "J0" (id 0) (at 62.23 59.69 0))
+    (property "Value" "VCC" (id 1) (at 55.88 59.69 0))
+    (property "Footprint" "Connector_Wire:SolderWirePad_1x01_SMD_1x2mm" (id 2) (at 64.77 59.69 0)
+      (effects (font (size 1.27 1.27)) hide)
+    )
+    (property "Datasheet" "~" (id 3) (at 64.77 59.69 0)
       (effects (font (size 1.27 1.27)) hide)
     )
@@
   )
   (symbol (lib_id "Connector:Conn_01x01_Male") (at 64.77 77.47 0) (unit 1)
-    (in_bom yes) (on_board yes)
+    (in_bom no) (on_board yes)
     (property "Reference" "J3" (id 0) (at 62.23 77.47 0))
     (property "Value" "GELB" (id 1) (at 55.88 77.47 0))
@@
   )
   (symbol (lib_id "Connector:Conn_01x01_Male") (at 64.77 81.28 0) (unit 1)
-    (in_bom yes) (on_board yes)
+    (in_bom no) (on_board yes)
     (property "Reference" "J4" (id 0) (at 62.23 81.28 0))
     (property "Value" "GRÜN" (id 1) (at 55.88 81.28 0))
@@
   )
   (symbol (lib_id "Connector:Conn_01x01_Male") (at 64.77 85.09 0) (unit 1)
-    (in_bom yes) (on_board yes)
+    (in_bom no) (on_board yes)
     (property "Reference" "J5" (id 0) (at 62.23 85.09 0))
     (property "Value" "Zs7-3" (id 1) (at 55.88 85.09 0))
@@
   )
   (symbol (lib_id "Connector:Conn_01x01_Male") (at 64.77 73.66 0) (unit 1)
-    (in_bom yes) (on_board yes)
+    (in_bom no) (on_board yes)
     (property "Reference" "J2" (id 0) (at 62.23 73.66 0))
     (property "Value" "ROT" (id 1) (at 55.88 73.66 0))

Commit message: MS: try using JLCPCB parts from library
Assign some LEDs available in JLCPCB's inhouse catalog.
Parts:
- D1, D10, D7: LCSC (none) -> C268305
- D2: LCSC (none) -> C268298
- D3: LCSC (none) -> C268302
- D5, D6, D8, D9: LCSC (none) -> C268299
Changed lines of the file:
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@@
+      (effects (font (size 1.27 1.27)) hide)
+    )
+    (property "LCSC" "C268299" (id 4) (at 151.13 63.8174 0)
       (effects (font (size 1.27 1.27)) hide)
     )
@@
       (effects (font (size 1.27 1.27)) hide)
     )
+    (property "LCSC" "C268299" (id 4) (at 128.27 63.8174 0)
+      (effects (font (size 1.27 1.27)) hide)
+    )
     (pin "1")
     (pin "2")
@@
     )
     (property "Datasheet" "~" (id 3) (at 170.18 63.5 0)
+      (effects (font (size 1.27 1.27)) hide)
+    )
+    (property "LCSC" "C268305" (id 4) (at 173.99 63.8174 0)
       (effects (font (size 1.27 1.27)) hide)
     )
@@
       (effects (font (size 1.27 1.27)) hide)
     )
+    (property "LCSC" "C268299" (id 4) (at 162.56 63.8174 0)
+      (effects (font (size 1.27 1.27)) hide)
+    )
     (pin "1")
     (pin "2")
@@
       (effects (font (size 1.27 1.27)) hide)
     )
+    (property "LCSC" "C268299" (id 4) (at 105.41 63.8174 0)
+      (effects (font (size 1.27 1.27)) hide)
+    )
     (pin "1")
     (pin "2")
@@
     )
     (property "Datasheet" "~" (id 3) (at 78.74 63.5 0)
+      (effects (font (size 1.27 1.27)) hide)
+    )
+    (property "LCSC" "C268305" (id 4) (at 82.55 63.8174 0)
       (effects (font (size 1.27 1.27)) hide)
     )
@@
       (effects (font (size 1.27 1.27)) hide)
     )
+    (property "LCSC" "C268302" (id 4) (at 116.84 63.8174 0)
+      (effects (font (size 1.27 1.27)) hide)
+    )
     (pin "1")
     (pin "2")
@@
     )
     (property "Datasheet" "~" (id 3) (at 135.89 63.5 0)
+      (effects (font (size 1.27 1.27)) hide)
+    )
+    (property "LCSC" "C268305" (id 4) (at 139.7 63.8174 0)
       (effects (font (size 1.27 1.27)) hide)
     )
@@
       (effects (font (size 1.27 1.27)) hide)
     )
+    (property "LCSC" "C268298" (id 4) (at 93.98 63.8174 0)
+      (effects (font (size 1.27 1.27)) hide)
+    )

Commit message: Update LCSC part numbers in schema
Parts:
- D1, D10, D7: LCSC C268305 -> C189305
- D2: LCSC C268298 -> C779449
- D3: LCSC C268302 -> C409787
- D5, D6, D8, D9: LCSC C268299 -> C779450
