File: kicad/Vorsignal/Vorsignal.kicad_pcb (KiCad board)
At the start: 2 copper layers, 6.6 x 10.8 mm, 7 parts, among them J0 VCC, J1 VkzBw, J3 GELB, J4 GRÜN

Commit message: Add CC-BY-SA 4.0 license
Parts:
- moved D3 25.5 mm to (98.6, 70.1)
- moved D5 25.5 mm to (102.0, 70.1)
- moved J0 25.5 mm to (102.4, 67.1)
- moved J3 25.5 mm to (98.5, 68.1)
- moved J4 25.5 mm to (98.5, 69.6)
- moved D1 25.5 mm to (98.6, 66.7)
- moved J1 25.5 mm to (98.5, 66.4)

Commit message: feat(VS): Add pre-signal repeater light
Parts:
- added D10: LED_W, LED_SMD:LED_0402_1005Metric, F.Cu at (98.4, 73.5)
- added J9: Wd, Connector_Wire:SolderWirePad_1x01_SMD_1x2mm, B.Cu at (98.5, 71.4)
Routing:
- net Net-(D10-K): track 0.00 -> 3.96 mm, vias 0 -> 1
- net Net-(D1-A): track 11.4 -> 13.9 mm
Other:
- board text added: "9"
- board text added: "VS v2"
- board text removed: "VSv1"
Changed lines of the file:
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@@
   (title_block
     (title "KS-Vorsignal")
-    (date "2023-12-17")
-    (rev "v1")
+    (date "2024-01-07")
+    (rev "2.0")
   )
   (layers
@@
   (net 3 "Net-(D3-K)")
   (net 4 "Net-(D5-K)")
+  (net 5 "Net-(D10-K)")
   (footprint "LED_SMD:LED_0402_1005Metric" locked (layer "F.Cu")
     (at 102 70.1 -90)
@@
     (descr "LED SMD 0402 (1005 Metric), square (rectangular) end terminal, IPC_7351 nominal, (Body size source: http://www.tortai-tech.com/upload/download/2011102023233369053.pdf), generated with kicad-footprint-generator")
     (tags "LED")
-    (property "LCSC" "C268305")
+    (property "LCSC" "C189305")
     (property "Sheetfile" "Vorsignal.kicad_sch")
     (property "Sheetname" "")
@@
     )
   )
+  (footprint "LED_SMD:LED_0402_1005Metric" (layer "F.Cu")
+    (at 98.4 73.5 90)
+    (descr "LED SMD 0402 (1005 Metric), square (rectangular) end terminal, IPC_7351 nominal, (Body size source: http://www.tortai-tech.com/upload/download/2011102023233369053.pdf), generated with kicad-footprint-generator")
+    (tags "LED")
+    (property "LCSC" "C189305")
+    (property "Sheetfile" "Vorsignal.kicad_sch")
+    (property "Sheetname" "")
+    (property "ki_description" "Light emitting diode")
+    (property "ki_keywords" "LED diode")
+    (attr smd)
+    (fp_text reference "D10" (at 0 -1.17 90) (layer "F.SilkS") hide
+        (effects (font (size 1 1) (thickness 0.15)))
+    )
+    (fp_text value "LED_W" (at 0 1.17 90) (layer "F.Fab")
+        (effects (font (size 1 1) (thickness 0.15)))
+    )
+    (fp_text user "${REFERENCE}" (at 0 0 90) (layer "F.Fab")
+        (effects (font (size 0.25 0.25) (thickness 0.04)))
+    )
+    (fp_circle (center -1.09 0) (end -1.04 0)
+      (stroke (width 0.1) (type solid)) (fill none) (layer "F.SilkS"))
+    (fp_line (start -0.93 -0.47) (end 0.93 -0.47)
+      (stroke (width 0.05) (type solid)) (layer "F.CrtYd"))
+    (fp_line (start -0.93 0.47) (end -0.93 -0.47)
+      (stroke (width 0.05) (type solid)) (layer "F.CrtYd"))
+    (fp_line (start 0.93 -0.47) (end 0.93 0.47)
+      (stroke (width 0.05) (type solid)) (layer "F.CrtYd"))
+    (fp_line (start 0.93 0.47) (end -0.93 0.47)
+      (stroke (width 0.05) (type solid)) (layer "F.CrtYd"))
+    (fp_line (start -0.5 -0.25) (end 0.5 -0.25)
+      (stroke (width 0.1) (type solid)) (layer "F.Fab"))
+    (fp_line (start -0.5 0.25) (end -0.5 -0.25)
+      (stroke (width 0.1) (type solid)) (layer "F.Fab"))
+    (fp_line (start -0.4 0.25) (end -0.4 -0.25)
+      (stroke (width 0.1) (type solid)) (layer "F.Fab"))
+    (fp_line (start -0.3 0.25) (end -0.3 -0.25)
+      (stroke (width 0.1) (type solid)) (layer "F.Fab"))
+    (fp_line (start 0.5 -0.25) (end 0.5 0.25)
+      (stroke (width 0.1) (type solid)) (layer "F.Fab"))
+    (fp_line (start 0.5 0.25) (end -0.5 0.25)
+      (stroke (width 0.1) (type solid)) (layer "F.Fab"))
+    (pad "1" smd roundrect (at -0.485 0 90) (size 0.59 0.64) (layers "F.Cu" "F.Paste" "F.Mask") (roundrect_rratio 0.25)
+      (net 5 "Net-(D10-K)") (pinfunction "K") (pintype "passive"))
+    (pad "2" smd roundrect (at 0.485 0 90) (size 0.59 0.64) (layers "F.Cu" "F.Paste" "F.Mask") (roundrect_rratio 0.25)
+      (net 2 "Net-(D1-A)") (pinfunction "A") (pintype "passive"))
+    (model "${KICAD6_3DMODEL_DIR}/LED_SMD.3dshapes/LED_0402_1005Metric.wrl"
+      (offset (xyz 0 0 0))
+      (scale (xyz 1 1 1))
+      (rotate (xyz 0 0 0))
+    )
+  )
   (footprint "LED_SMD:LED_0402_1005Metric" locked (layer "F.Cu")
     (at 98.6 70.1 -90)
@@
   )
   (footprint "Connector_Wire:SolderWirePad_1x01_SMD_1x2mm" (layer "B.Cu")
+    (at 98.5 71.4 90)
+    (descr "Wire Pad, Square, SMD Pad,  1mm x 2mm,")
+    (tags "MesurementPoint Square SMDPad 1mmx2mm ")
+    (property "Sheetfile" "Vorsignal.kicad_sch")
+    (property "Sheetname" "")
+    (property "exclude_from_bom" "")
+    (property "ki_description" "Generic connector, single row, 01x01, script generated (kicad-library-utils/schlib/autogen/connector/)")
+    (property "ki_keywords" "connector")
+    (attr exclude_from_pos_files exclude_from_bom)
+    (fp_text reference "J9" (at 0 2.54 90) (layer "B.SilkS") hide
+        (effects (font (size 1 1) (thickness 0.15)) (justify mirror))
+    )
+    (fp_text value "Wd" (at 0 -2.54 90) (layer "B.Fab")
+        (effects (font (size 1 1) (thickness 0.15)) (justify mirror))
+    )
+    (fp_text user "${REFERENCE}" (at 0 0 90) (layer "B.Fab")
+        (effects (font (size 1 1) (thickness 0.15)) (justify mirror))
+    )
+    (fp_line (start -0.63 -1.27) (end 0.63 -1.27)
+      (stroke (width 0.05) (type solid)) (layer "B.CrtYd"))
+    (fp_line (start -0.63 1.27) (end -0.63 -1.27)
+      (stroke (width 0.05) (type solid)) (layer "B.CrtYd"))
+    (fp_line (start 0.63 -1.27) (end 0.63 1.27)
+      (stroke (width 0.05) (type solid)) (layer "B.CrtYd"))
+    (fp_line (start 0.63 1.27) (end -0.63 1.27)
+      (stroke (width 0.05) (type solid)) (layer "B.CrtYd"))
+    (fp_line (start -0.63 -1.27) (end -0.63 1.27)
+      (stroke (width 0.1) (type solid)) (layer "B.Fab"))
+    (fp_line (start -0.63 1.27) (end 0.63 1.27)
+      (stroke (width 0.1) (type solid)) (layer "B.Fab"))
+    (fp_line (start 0.63 -1.27) (end -0.63 -1.27)
+      (stroke (width 0.1) (type solid)) (layer "B.Fab"))
+    (fp_line (start 0.63 1.27) (end 0.63 -1.27)
+      (stroke (width 0.1) (type solid)) (layer "B.Fab"))
+    (pad "1" smd roundrect (at 0 0 90) (size 1 2) (layers "B.Cu" "B.Paste" "B.Mask") (roundrect_rratio 0.25)
+      (net 5 "Net-(D10-K)") (pinfunction "Pin_1") (pintype "passive"))
+  )
+  (footprint "Connector_Wire:SolderWirePad_1x01_SMD_1x2mm" (layer "B.Cu")
     (at 98.5 68.1 -90)
     (descr "Wire Pad, Square, SMD Pad,  5mm x 10mm,")
@@
   )
   (gr_line (start 98.6 70.1) (end 100.3 70.1)
+    (stroke (width 0.1) (type default)) (layer "Dwgs.User"))
+  (gr_line (start 100.3 73.5) (end 98.4 73.5)
     (stroke (width 0.1) (type default)) (layer "Dwgs.User"))
   (gr_line (start 100.3 70.1) (end 100.3 64.7)
@@
   (gr_line (start 100.3 75.5) (end 100.3 70.1)
     (stroke (width 0.1) (type default)) (layer "Dwgs.User"))
-  (gr_line (start 100.3 73.5) (end 98.6 73.5)
-    (stroke (width 0.1) (type default)) (layer "Dwgs.User"))
   (gr_arc (start 103.6 75) (mid 103.453553 75.353553) (end 103.1 75.5)
     (stroke (width 0.0381) (type solid)) (layer "Edge.Cuts"))
@@
   (gr_arc (start 97 65.2) (mid 97.146447 64.846447) (end 97.5 64.7)
     (stroke (width 0.0381) (type solid)) (layer "Edge.Cuts"))
+  (gr_text "9" (at 100.3 71.4) (layer "B.SilkS")
+    (effects (font (size 0.8128 0.8128) (thickness 0.1524)) (justify mirror))
+  )
   (gr_text "1" (at 100.3 66.4) (layer "B.SilkS")
     (effects (font (size 0.8128 0.8128) (thickness 0.1524)) (justify mirror))
@@
     (effects (font (size 0.8128 0.8128) (thickness 0.1524)) (justify mirror))
   )
-  (gr_text "VSv1" (at 100.3 74.5) (layer "B.SilkS")
+  (gr_text "VS v2" (at 100.3 74.5) (layer "B.SilkS")
     (effects (font (size 1 1) (thickness 0.1524)) (justify mirror))
   )
@@
   (segment (start 99.2 67.1) (end 98.5 66.4) (width 0.2) (layer "B.Cu") (net 1))
   (segment (start 99.8 67.1) (end 99.2 67.1) (width 0.2) (layer "B.Cu") (net 1))
+  (segment (start 100.7 67.8) (end 100.7 70.585) (width 0.2) (layer "F.Cu") (net 2))
+  (segment (start 100.7 70.585) (end 102 70.585) (width 0.2) (layer "F.Cu") (net 2))
+  (segment (start 98.6 71.7) (end 98.4 71.9) (width 0.2) (layer "F.Cu") (net 2))
   (segment (start 101.4 67.1) (end 100.7 67.8) (width 0.2) (layer "F.Cu") (net 2))
-  (segment (start 100.7 70.6) (end 100.715 70.585) (width 0.2) (layer "F.Cu") (net 2))
+  (segment (start 98.6 70.585) (end 100.7 70.585) (width 0.2) (layer "F.Cu") (net 2))
   (segment (start 98.6 66.215) (end 100.515 66.215) (width 0.2) (layer "F.Cu") (net 2))
+  (segment (start 98.6 70.585) (end 98.6 71.7) (width 0.2) (layer "F.Cu") (net 2))
   (segment (start 100.515 66.215) (end 101.4 67.1) (width 0.2) (layer "F.Cu") (net 2))
-  (segment (start 100.7 67.8) (end 100.7 70.6) (width 0.2) (layer "F.Cu") (net 2))
-  (segment (start 100.715 70.585) (end 98.6 70.585) (width 0.2) (layer "F.Cu") (net 2))
-  (segment (start 100.715 70.585) (end 102 70.585) (width 0.2) (layer "F.Cu") (net 2))
+  (segment (start 98.4 71.9) (end 98.4 73.015) (width 0.2) (layer "F.Cu") (net 2))
   (via (at 101.4 67.1) (size 0.6) (drill 0.3) (layers "F.Cu" "B.Cu") (net 2))
   (segment (start 101.4 67.1) (end 102.4 67.1) (width 0.2) (layer "B.Cu") (net 2))
@@
   (via (at 101.4 68.1) (size 0.6) (drill 0.3) (layers "F.Cu" "B.Cu") (net 4))
   (segment (start 101.4 68.1) (end 98.5 68.1) (width 0.2) (layer "B.Cu") (net 4))
+  (segment (start 98.4 73.985) (end 99.115 73.985) (width 0.2) (layer "F.Cu") (net 5))
+  (segment (start 99.115 73.985) (end 99.6 73.5) (width 0.2) (layer "F.Cu") (net 5))
+  (via (at 99.6 73.5) (size 0.6) (drill 0.3) (layers "F.Cu" "B.Cu") (net 5))
+  (segment (start 99.6 72.5) (end 98.5 71.4) (width 0.2) (layer "B.Cu") (net 5))
+  (segment (start 99.6 73.5) (end 99.6 72.5) (width 0.2) (layer "B.Cu") (net 5))
 )
